Commit message: Add Gazebo Specific Tag to Robot URDF & Gazebo World Launch file

File: Project_2/shady_ws/src/shady_description/urdf/shady.urdf (robot description, URDF)
Before this commit: robot shady, 3 links, 2 joints
Links:
- link base_link: mass None -> 8
- link left_wheel: mass None -> 0.3; geometry collision cylinder length=0.1 radius=0.15; visual cylinder length=0.1 radius=0.15
- link right_wheel: mass None -> 0.3; geometry collision cylinder length=0.1 radius=0.15; visual cylinder length=0.1 radius=0.15

Commit message: Add Hokuyo Laser Gazebo Plugin

File: Project_2/shady_ws/src/shady_description/urdf/shady.urdf (robot description, URDF)
Before this commit: robot shady, 3 links, 2 joints
Links:
- added link hokuyo_link, mass 1e-5; collision box size=0.1 0.1 0.1; visual mesh filename=package://shady_description/hokuyo/meshes/hokuyo.dae
Joints:
- added joint hokuyo_joint: type fixed, parent base_link, child hokuyo_link, origin xyz=0.3 0 0.15 rpy=0 0 0, axis 0 1 0
